File: Labo7/simulador/Kicad/amplificador_programable/version_final/amplificador_programable.kicad_pcb_3.kicad_pcb (KiCad board)
At the start: 2 copper layers, 86.5 x 65 mm, 13 parts, among them J1 Conn_Coaxial, J2 Conn_02x06_Counter_Clockwise, J3 Conn_Coaxial, SW1 SW_DIP_x04, U1 TL072, U2 INA110KP

Commit message: data simulacion
Parts:
- moved J2 9.96 mm to (121.9, 96.5)
- moved C3 3.01 mm to (125.8, 74.8)
- moved C4 2.76 mm to (131.5, 74.8)
Routing:
- net VCC: track 41.3 -> 52.5 mm
- net Net-(U2-G=10): track 29.3 -> 38.6 mm
- net Net-(U2-G=100): track 29.2 -> 37.4 mm
- net Net-(U2-G=500): track 26.2 -> 34.3 mm
- net Net-(U2-G=200): track 27.8 -> 31.8 mm
- net VDD: track 60.3 -> 62.2 mm
